Commit message: sim README 对齐当前默认（geometric/零位 init_pose）+ joint3/5 限位放宽全链一致
- astral_mujoco_sim README：默认求解器 urdf_numerical→geometric、init_pose 改述为 yaml 零位覆盖、MJCF 表补 mjcf_path 回退
- joint3/5 限位 ±1.57 → ±2.2689/±1.7802：astral_arm(.pin).urdf、astral_robot(.pin).urdf、内嵌 RobotMain_URDF.pin.urdf、astral_dual.xml（range+ctrlrange）、analytic.py
- test_geometric_ik 满伸 sweep：>0.15 rad 跳变仅当 esc_active 放行（分支逃逸设计），无逃逸跳变仍 FAIL

Co-authored-by: Cursor <cursoragent@cursor.com>

File: src/astral_arm_description/urdf/astral_arm.pin.urdf (robot description, URDF)
Before this commit: robot astral_arm, 9 links, 8 joints
Joints:
- joint joint3: limit lower=-1.57 upper=1.57 effort=100 velocity=10 -> lower=-2.2689 upper=2.2689 effort=100 velocity=10
- joint joint5: limit lower=-1.57 upper=1.57 effort=100 velocity=10 -> lower=-1.7802 upper=1.7802 effort=100 velocity=10

File: src/astral_arm_teleop/astral_arm_teleop/robot/urdf/RobotMain_URDF.pin.urdf (robot description, URDF)
Before this commit: robot RobotMain_URDF, 15 links, 14 joints
Joints:
- joint Joint_la_3: limit lower=-1.57 upper=1.57 effort=100 velocity=10 -> lower=-2.2689 upper=2.2689 effort=100 velocity=10
- joint Joint_la_5: limit lower=-1.57 upper=1.57 effort=100 velocity=10 -> lower=-1.7802 upper=1.7802 effort=100 velocity=10
- joint Joint_ra_3: limit lower=-1.57 upper=1.57 effort=100 velocity=10 -> lower=-2.2689 upper=2.2689 effort=100 velocity=10
- joint Joint_ra_5: limit lower=-1.57 upper=1.57 effort=100 velocity=10 -> lower=-1.7802 upper=1.7802 effort=100 velocity=10

File: src/astral_robot_description/urdf/astral_robot.pin.urdf (robot description, URDF)
Before this commit: robot astral_robot, 18 links, 17 joints
Joints:
- joint left_joint3: limit lower=-1.57 upper=1.57 effort=100 velocity=10 -> lower=-2.2689 upper=2.2689 effort=100 velocity=10
- joint left_joint5: limit lower=-1.57 upper=1.57 effort=100 velocity=10 -> lower=-1.7802 upper=1.7802 effort=100 velocity=10
- joint right_joint3: limit lower=-1.57 upper=1.57 effort=100 velocity=10 -> lower=-2.2689 upper=2.2689 effort=100 velocity=10
- joint right_joint5: limit lower=-1.57 upper=1.57 effort=100 velocity=10 -> lower=-1.7802 upper=1.7802 effort=100 velocity=10
